Commit message: -

File: urdf/tb3.urdf.xacro (robot description, xacro)
@@ -3,5 +3,5 @@
   <xacro:include filename="$(find rl_tb3)/urdf/tb3commprop.xacro"/>
   <xacro:include filename="$(find rl_tb3)/urdf/tb3.gazebo.xacro"/>
-  <xacro:include filename="$(find realsense2_description)/urdf/_materials.urdf.xacro" />
+  <!-- <xacro:include filename="$(find realsense2_description)/urdf/_materials.urdf.xacro" /> -->
   <xacro:property name="M_PI" value="3.1415926535897931" />
   <xacro:property name="d455_cam_depth_to_infra1_offset" value="0.0"/>
@@ -151,5 +151,5 @@
       <geometry>
         <!-- <box size="${d455_cam_depth} ${d455_cam_width} ${d455_cam_height}"/> -->
-        <mesh filename="package://realsense2_description/meshes/d455.stl" scale="0.001 0.001 0.001" />
+        <mesh filename="package://rl_tb3/meshes/d455.stl" scale="0.001 0.001 0.001" />
       </geometry>
       <material name="aluminum"/>

File: urdf/tb3commprop.xacro (robot description, xacro)
@@ -32,3 +32,6 @@
     <color rgba="1.0 1.0 1.0 1.0"/>
   </material>
+  <material name='aluminum'>
+    <color rgba = "${189/255} ${189/255} ${189/255} 1.0"/>
+  </material>
 </robot>
